File: PCB/guilty-devboard-idk.kicad_sch (KiCad schematic)
At the start: 56 parts, among them J1 USB_C_Receptacle_USB2.0_16P, Q1 SP2038CNQ, U1 nRF54LM20A-QGAA, U2 SGM40567-4.2XG/TR, U3 Xiao nRF52840 Connectors, U4 TCA9536, U5 FH9261-G3JH, U6 BD83070GWL-E2, Y1 32MHz, Y2 32.768kHz

Commit message: fix pads being slightly off, should now match xiao pretty much perfectly
Parts:
- U3: value Xiao nRF52840 Connectors -> (none)
Changed lines of the file:
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@@
 	)
 	(symbol
-		(lib_id "guilty-devboard:Guilty Devboard Xrd Connectors (dev)")
-		(at 133.35 265.43 0)
-		(unit 1)
-		(body_style 1)
-		(exclude_from_sim no)
-		(in_bom no)
-		(on_board yes)
-		(in_pos_files yes)
-		(dnp no)
-		(fields_autoplaced yes)
-		(property "Reference" "U3"
-			(at 123.19 296.418 0)
-			(hide yes)
-			(show_name no)
-			(do_not_autoplace no)
-			(effects
-				(font
-					(size 1.27 1.27)
-				)
-			)
-		)
-		(property "Value" "Xiao nRF52840 Connectors"
-			(at 123.19 298.958 0)
-			(hide yes)
-			(show_name no)
-			(do_not_autoplace no)
-			(effects
-				(font
-					(size 1.27 1.27)
-				)
-			)
-		)
-		(property "Footprint" "guilty-devboard-idk:Guilty Devboard Xrd pads"
-			(at 133.35 314.198 0)
-			(hide yes)
-			(show_name no)
-			(do_not_autoplace no)
-			(effects
-				(font
-					(size 1.27 1.27)
-				)
-			)
-		)
-		(property "Datasheet" ""
-			(at 120.65 251.46 0)
-			(hide yes)
-			(show_name no)
-			(do_not_autoplace no)
-			(effects
-				(font
-					(size 1.27 1.27)
-				)
-			)
-		)
-		(property "Description" "Symbol for a Seeeduino Xiao nRF52840 Plus"
-			(at 133.35 265.43 0)
-			(hide yes)
-			(show_name no)
-			(do_not_autoplace no)
-			(effects
-				(font
-					(size 1.27 1.27)
-				)
-			)
-		)
-		(pin "21"
-		)
-		(pin "7"
-		)
-		(pin "5"
-		)
-		(pin "4"
-		)
-		(pin "3"
-		)
-		(pin "2"
-		)
-		(pin "1"
-		)
-		(pin "6"
-		)
-		(pin "23"
-		)
-		(pin "10"
-		)
-		(pin "30"
-		)
-		(pin "28"
-		)
-		(pin "34"
-		)
-		(pin "26"
-		)
-		(pin "36"
-		)
-		(pin "9"
-		)
-		(pin "31"
-		)
-		(pin "35"
-		)
-		(pin "8"
-		)
-		(pin "22"
-		)
-		(pin "17"
-		)
-		(pin "27"
-		)
-		(pin "11"
-		)
-		(pin "13"
-		)
-		(pin "25"
-		)
-		(pin "33"
-		)
-		(pin "12"
-		)
-		(pin "16"
-		)
-		(pin "32"
-		)
-		(pin "15"
-		)
-		(pin "14"
-		)
-		(pin "24"
-		)
-		(pin "19"
-		)
-		(pin "20"
-		)
-		(pin "18"
-		)
-		(pin "29"
-		)
-		(instances
-			(project "guilty-devboard-idk"
-				(path "/f655de09-440b-4c8a-8451-7845142cd85d"
-					(reference "U3")
-					(unit 1)
-				)
-			)
-		)
-	)
-	(symbol
 		(lib_id "KiCad:C_Small")
 		(at 109.22 46.99 0)
@@
 					(unit 1)
 				)
+			)
+		)
+	)
+	(symbol
+		(lib_id "guilty-devboard:Guilty Devboard Xrd Connectors (dev)")
+		(at 133.35 265.43 0)
+		(unit 1)
+		(body_style 1)
+		(exclude_from_sim no)
+		(in_bom no)
+		(on_board yes)
+		(in_pos_files yes)
+		(dnp no)
+		(fields_autoplaced yes)
+		(property "Reference" "U3"
+			(at 123.19 296.418 0)
+			(hide yes)
+			(show_name no)
+			(do_not_autoplace no)
+			(effects
+				(font
+					(size 1.27 1.27)
+				)
+			)
+		)
+		(property "Value" ""
+			(at 123.19 298.958 0)
+			(hide yes)
+			(show_name no)
+			(do_not_autoplace no)
+			(effects
+				(font
+					(size 1.27 1.27)
+				)
+			)
+		)
+		(property "Footprint" "guilty-devboard-idk:Guilty Devboard Xrd pads"
+			(at 133.35 314.198 0)
+			(hide yes)
+			(show_name no)
+			(do_not_autoplace no)
+			(effects
+				(font
+					(size 1.27 1.27)
+				)
+			)
+		)
+		(property "Datasheet" ""
+			(at 120.65 251.46 0)
+			(hide yes)
+			(show_name no)
+			(do_not_autoplace no)
+			(effects
+				(font
+					(size 1.27 1.27)
+				)
+			)
+		)
+		(property "Description" "Symbol for Guilty Devboard Xrd development"
+			(at 133.35 265.43 0)
+			(hide yes)
+			(show_name no)
+			(do_not_autoplace no)
+			(effects
+				(font
+					(size 1.27 1.27)
+				)
+			)
+		)
+		(pin "32"
+		)
+		(pin "18"
+		)
+		(pin "16"
+		)
+		(pin "30"
+		)
+		(pin "21"
+		)
+		(pin "15"
+		)
+		(pin "14"
+		)
+		(pin "13"
+		)
+		(pin "12"
+		)
+		(pin "11"
+		)
+		(pin "35"
+		)
+		(pin "28"
+		)
+		(pin "36"
+		)
+		(pin "25"
+		)
+		(pin "10"
+		)
+		(pin "9"
+		)
+		(pin "8"
+		)
+		(pin "7"
+		)
+		(pin "6"
+		)
+		(pin "5"
+		)
+		(pin "4"
+		)
+		(pin "3"
+		)
+		(pin "2"
+		)
+		(pin "1"
+		)
+		(pin "19"
+		)
+		(pin "23"
+		)
+		(pin "22"
+		)
+		(pin "24"
+		)
+		(pin "29"
+		)
+		(pin "17"
+		)
+		(pin "26"
+		)
+		(pin "34"
+		)
+		(pin "33"
+		)
+		(pin "27"
+		)
+		(pin "31"
+		)
+		(pin "20"
+		)
+		(instances
+			(project "guilty-devboard-idk"
+				(path "/f655de09-440b-4c8a-8451-7845142cd85d"
+					(reference "U3")
+					(unit 1)
+				)
